File: kicad/at2usb_jp/at2usb_jp.kicad_sch (KiCad schematic)
At the start: 4 parts, among them J1 USB_B, U1 PIC16F1455

Commit message: update
Connections:
- net GND: now also C1.2
Changed lines of the file:
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@@
 	(symbol
 		(lib_id "power:GND")
-		(at 43.18 36.83 0)
+		(at 43.18 33.02 0)
 		(unit 1)
 		(exclude_from_sim no)
@@
 		(fields_autoplaced yes)
 		(property "Reference" "#PWR01"
-			(at 43.18 43.18 0)
+			(at 43.18 39.37 0)
 			(effects
 				(font
@@
 		)
 		(property "Value" "GND"
-			(at 43.18 41.91 0)
+			(at 43.18 38.1 0)
 			(effects
 				(font
@@
 		)
 		(property "Footprint" ""
-			(at 43.18 36.83 0)
+			(at 43.18 33.02 0)
 			(effects
 				(font
@@
 		)
 		(property "Datasheet" ""
-			(at 43.18 36.83 0)
+			(at 43.18 33.02 0)
 			(effects
 				(font
@@
 		)
 		(property "Description" "Power symbol creates a global label with name \"GND\" , ground"
-			(at 43.18 36.83 0)
+			(at 43.18 33.02 0)
 			(effects
 				(font
